File: STM32-FC/schematic/io_communication.kicad_sch (KiCad schematic)
At the start: 38 parts, among them J10 SM06B-GHS-TBT, J11 SM06B-GHS-TBT, J12 PWM_Conn_3x14, J13 SM04B-GHS-TBT, J14 ZH 1.5mm 4P, J15 SM06B-GHS-TBT, J5 SM06B-GHS-TBT, J6 SM06B-GHS-TBT, J7 SM04B-GHS-TBT, J8 SM04B-GHS-TBT, J9 SM04B-GHS-TBT, Q1 PMDPB30XN, U11 ATA6561-GBQW, U12 ATA6561-GBQW, U13 TMUX1104

Commit message: init:footprint
footprint 작업 시작
Parts:
- J10, J11, J5, J6: footprint JST_GH:JST_GH_SM06B-GHS-TB_06x1.25mm_Angled -> Connector_JST:JST_GH_SM06B-GHS-TB_1x06-1MP_P1.25mm_Horizontal
- J13, J7, J8, J9: footprint JST_GH:JST_GH_SM04B-GHS-TB_04x1.25mm_Angled -> Connector_JST:JST_GH_SM04B-GHS-TB_1x04-1MP_P1.25mm_Horizontal
- J15: footprint (none) -> Connector_JST:JST_GH_SM06B-GHS-TB_1x06-1MP_P1.25mm_Horizontal
Changed lines of the file:
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@@
 			)
 		)
-		(property "Footprint" "JST_GH:JST_GH_SM06B-GHS-TB_06x1.25mm_Angled"
+		(property "Footprint" "Connector_JST:JST_GH_SM06B-GHS-TB_1x06-1MP_P1.25mm_Horizontal"
 			(at 63.5 36.83 0)
 			(effects
@@
 			)
 		)
-		(property "Footprint" ""
+		(property "Footprint" "Connector_JST:JST_GH_SM06B-GHS-TB_1x06-1MP_P1.25mm_Horizontal"
 			(at 203.2 146.05 0)
 			(effects
@@
 			)
 		)
-		(property "Footprint" "JST_GH:JST_GH_SM04B-GHS-TB_04x1.25mm_Angled"
+		(property "Footprint" "Connector_JST:JST_GH_SM04B-GHS-TB_1x04-1MP_P1.25mm_Horizontal"
 			(at 154.94 127 0)
 			(effects
@@
 			)
 		)
-		(property "Footprint" "JST_GH:JST_GH_SM06B-GHS-TB_06x1.25mm_Angled"
+		(property "Footprint" "Connector_JST:JST_GH_SM06B-GHS-TB_1x06-1MP_P1.25mm_Horizontal"
 			(at 113.03 104.14 0)
 			(effects
@@
 			)
 		)
-		(property "Footprint" "JST_GH:JST_GH_SM04B-GHS-TB_04x1.25mm_Angled"
+		(property "Footprint" "Connector_JST:JST_GH_SM04B-GHS-TB_1x04-1MP_P1.25mm_Horizontal"
 			(at 63.5 104.14 0)
 			(effects
@@
 			)
 		)
-		(property "Footprint" "JST_GH:JST_GH_SM04B-GHS-TB_04x1.25mm_Angled"
+		(property "Footprint" "Connector_JST:JST_GH_SM04B-GHS-TB_1x04-1MP_P1.25mm_Horizontal"
 			(at 104.14 180.34 0)
 			(effects
@@
 			)
 		)
-		(property "Footprint" "JST_GH:JST_GH_SM06B-GHS-TB_06x1.25mm_Angled"
+		(property "Footprint" "Connector_JST:JST_GH_SM06B-GHS-TB_1x06-1MP_P1.25mm_Horizontal"
 			(at 63.5 73.66 0)
 			(effects
@@
 			)
 		)
-		(property "Footprint" "JST_GH:JST_GH_SM06B-GHS-TB_06x1.25mm_Angled"
+		(property "Footprint" "Connector_JST:JST_GH_SM06B-GHS-TB_1x06-1MP_P1.25mm_Horizontal"
 			(at 113.03 49.53 0)
 			(effects
@@
 			)
 		)
-		(property "Footprint" "JST_GH:JST_GH_SM04B-GHS-TB_04x1.25mm_Angled"
+		(property "Footprint" "Connector_JST:JST_GH_SM04B-GHS-TB_1x04-1MP_P1.25mm_Horizontal"
 			(at 104.14 140.97 0)
 			(effects
