File: STM32-FC/schematic/usb.kicad_sch (KiCad schematic)
At the start: 27 parts, among them J2 USB_C_USB2.0_14P, J3 SM06B-GHS-TBT, U1 USBLC6-2SC6, U2 TPS62840, U3 TPS62840, U4 TPS62840

Commit message: init:footprint
footprint 작업 시작
Parts:
- J3: footprint JST_GH:JST_GH_SM06B-GHS-TB_06x1.25mm_Angled -> Connector_JST:JST_GH_SM06B-GHS-TB_1x06-1MP_P1.25mm_Horizontal
Changed lines of the file:
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@@
 			)
 		)
-		(property "Footprint" "JST_GH:JST_GH_SM06B-GHS-TB_06x1.25mm_Angled"
+		(property "Footprint" "Connector_JST:JST_GH_SM06B-GHS-TB_1x06-1MP_P1.25mm_Horizontal"
 			(at 215.9 50.8 0)
 			(effects
