File: STM32-FC/schematic/STM32_io.kicad_sch (KiCad schematic)
At the start: 33 parts, among them IC1 STM32F746NGH6, Q1 PMDPB30XN

Commit message: init:footprint
footprint 작업 시작
Parts:
- IC1: footprint BGA216C80P15X15_1300X1300X110 -> STM32F746NGH6:STM32F746NGH6
Changed lines of the file:
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@@
 			)
 		)
-		(property "Footprint" "BGA216C80P15X15_1300X1300X110"
+		(property "Footprint" "STM32F746NGH6:STM32F746NGH6"
 			(at 214.122 36.068 0)
 			(effects
@@
 			)
 		)
-		(property "Footprint" "BGA216C80P15X15_1300X1300X110"
+		(property "Footprint" "STM32F746NGH6:STM32F746NGH6"
 			(at 328.422 36.068 0)
 			(effects

Commit message: update : BOM and minor fix
- remove : DC2DC for analog
- change : JST SM conn. to BM
- change : ELRS conn. to JST XH (instead of JST SM)
- update : BOM List
Parts:
- IC1: LCSC (none) -> C503080
Changed lines of the file:
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@@
+			)
+		)
+		(property "LCSC" "C503080"
+			(at 85.09 91.44 0)
+			(effects
+				(font
+					(size 1.27 1.27)
+				)
+				(hide yes)
 			)
 		)
@@
 			(at 199.39 91.44 0)
 			(effects
+				(font
+					(size 1.27 1.27)
+				)
+				(hide yes)
+			)
+		)
+		(property "LCSC" "C503080"
+			(at 199.39 91.44 0)
+			(effects

Commit message: change : RC size 0402 to 0201
Parts:
- C10, C11, C12, C13, C14, C15, C17, C19, C20, C21, C22, C23, C24, C25, C26, C29: footprint Capacitor_SMD:C_0402_1005Metric -> Capacitor_SMD:C_0201_0603Metric; LCSC C1525 -> C49062
- C16, C18: footprint Capacitor_SMD:C_0402_1005Metric -> Capacitor_SMD:C_0201_0603Metric; LCSC C14445 -> C318542
- R2, R4, R5, R6: footprint Resistor_SMD:R_0402_1005Metric -> Resistor_SMD:R_0201_0603Metric; LCSC C25079 -> C295718
- R3, R7: footprint Resistor_SMD:R_0402_1005Metric -> Resistor_SMD:R_0201_0603Metric; LCSC C25531 -> C106225
