File: STM32-FC/schematic/io_GPS.kicad_sch (KiCad schematic)
At the start: 8 parts, among them J10 GH 1.25mm 6P, J9 GH 1.25mm 10P

Commit message: schematic update
Other:
- title: GPS -> STM32 Flight Controller
