File: STM32-FC/schematic/io_RC_INPUT.kicad_sch (KiCad schematic)
At the start: 9 parts, among them J6 PWM_Conn_3x14, J7 ZH 1.5mm 3P, J8 ZH 1.5mm 4P, Q2 S9013

Commit message: schematic update
Other:
- title: RC_INPUT -> STM32 Flight Controller
Changed lines of the file:
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@@
 (kicad_sch
-	(version 20231120)
+	(version 20250114)
 	(generator "eeschema")
-	(generator_version "8.0")
+	(generator_version "9.0")
 	(paper "A4")
 	(title_block
-		(title "RC_INPUT")
-		(date "2025-02-08")
-		(rev "A")
+		(title "STM32 Flight Controller")
+		(date "2025-09-16")
+		(rev "v1.0.0")
 		(company "NARAE")
 		(comment 1 "INHA Univ. Areo-modelling Club")
 		(comment 2 "2024 Winter UAV Project ")
 	)
+	(rectangle
+		(start 88.9 53.34)
+		(end 152.4 78.74)
+		(stroke
+			(width 0)
+			(type dash)
+		)
+		(fill
+			(type none)
+		)
+	)
+	(rectangle
+		(start 22.8481 12.6751)
+		(end 86.3481 116.84)
+		(stroke
+			(width 0)
+			(type dash)
+		)
+		(fill
+			(type none)
+		)
+	)
+	(rectangle
+		(start 88.9 12.7)
+		(end 152.4 50.8)
+		(stroke
+			(width 0)
+			(type dash)
+		)
+		(fill
+			(type none)
+		)
+	)
+	(rectangle
+		(start 88.9 81.28)
+		(end 152.4 116.84)
+		(stroke
+			(width 0)
+			(type dash)
+		)
+		(fill
+			(type none)
+		)
+	)
+	(text "RCIN (SBUS/PPM/SRXL2)"
+		(exclude_from_sim no)
+		(at 89.916 15.494 0)
+		(effects
+			(font
+				(size 1.27 1.27)
+			)
+			(justify left bottom)
+		)
+	)
+	(text "ZH 1.5mm 3P\n\nPA10 : USART1_RX"
+		(exclude_from_sim no)
+		(at 89.916 58.674 0)
+		(effects
+			(font
+				(size 1.27 1.27)
+			)
+			(justify left top)
+		)
+	)
+	(text "SRXL2"
+		(exclude_from_sim no)
+		(at 89.916 84.074 0)
+		(effects
+			(font
+				(size 1.27 1.27)
+			)
+			(justify left bottom)
+		)
+	)
+	(text "2.54mm 3P\n\nSBUS   : PA10 : USART1_RX\nPPM_IN : PD15 : TIM4_CH4\nSRXL2  : PA9  : USART1_TX\n"
+		(exclude_from_sim no)
+		(at 89.916 18.034 0)
+		(effects
+			(font
+				(size 1.27 1.27)
+			)
+			(justify left top)
+		)
+	)
+	(text "DSM"
+		(exclude_from_sim no)
+		(at 89.916 56.134 0)
+		(effects
+			(font
+				(size 1.27 1.27)
+			)
+			(justify left bottom)
+		)
+	)
+	(text "MAIN 1 : PA0 : TIM5_CH1\nMAIN 2 : PA1 : TIM5_CH2\nMAIN 3 : PA2 : TIM5_CH3\nMAIN 4 : PA3 : TIM5_CH4\nMAIN 5 : PC6 : TIM3_CH1\nMAIN 6 : PC7 : TIM3_CH2\nMAIN 7 : PB0 : TIM3_CH3\nMAIN 8 : PB1 : TIM3_CH4"
+		(exclude_from_sim no)
+		(at 23.8641 18.0091 0)
+		(effects
+			(font
+				(size 1.27 1.27)
+			)
+			(justify left top)
+		)
+	)
+	(text "PWM RC OUT"
+		(exclude_from_sim no)
+		(at 23.8641 15.4691 0)
+		(effects
+			(font
+				(size 1.27 1.27)
+			)
+			(justify left bottom)
+		)
+	)
+	(text "AUX1 : PB7 : TIM4_CH1\nAUX2 : PE11 : TIM1_CH2\nAUX3 : PE13 : TIM1_CH3\nAUX4 : PE14 : TIM1_CH4\n\nRCIN : PPM/SBUS/SRXL2\nRSSI_IN : PC1 : ADC123_IN11"
+		(exclude_from_sim no)
+		(at 23.8641 35.7891 0)
+		(effects
+			(font
+				(size 1.27 1.27)
+			)
+			(justify left top)
+		)
+	)
+	(text "ZH 1.5mm 4P\n\nPA9 : USART1_TX (Half Duplex)"
+		(exclude_from_sim no)
+		(at 89.916 86.614 0)
+		(effects
+			(font
+				(size 1.27 1.27)
+			)
+			(justify left top)
+		)
+	)
 	(junction
 		(at 118.11 39.37)
@@
 		)
 	)
-	(rectangle
-		(start 88.9 53.34)
-		(end 152.4 78.74)
-		(stroke
-			(width 0)
-			(type dash)
-		)
-		(fill
-			(type none)
-		)
-	)
-	(rectangle
-		(start 22.8481 12.6751)
-		(end 86.3481 116.84)
-		(stroke
-			(width 0)
-			(type dash)
-		)
-		(fill
-			(type none)
-		)
-	)
-	(rectangle
-		(start 88.9 12.7)
-		(end 152.4 50.8)
-		(stroke
-			(width 0)
-			(type dash)
-		)
-		(fill
-			(type none)
-		)
-	)
-	(rectangle
-		(start 88.9 81.28)
-		(end 152.4 116.84)
-		(stroke
-			(width 0)
-			(type dash)
-		)
-		(fill
-			(type none)
-		)
-	)
-	(text "RCIN (SBUS/PPM/SRXL2)"
-		(exclude_from_sim no)
-		(at 89.916 15.494 0)
-		(effects
-			(font
-				(size 1.27 1.27)
-			)
-			(justify left bottom)
-		)
-	)
-	(text "ZH 1.5mm 3P\n\nPA10 : USART1_RX"
-		(exclude_from_sim no)
-		(at 89.916 58.674 0)
-		(effects
-			(font
-				(size 1.27 1.27)
-			)
-			(justify left top)
-		)
-	)
-	(text "SRXL2"
-		(exclude_from_sim no)
-		(at 89.916 84.074 0)
-		(effects
-			(font
-				(size 1.27 1.27)
-			)
-			(justify left bottom)
-		)
-	)
-	(text "2.54mm 3P\n\nSBUS   : PA10 : USART1_RX\nPPM_IN : PD15 : TIM4_CH4\nSRXL2  : PA9  : USART1_TX\n"
-		(exclude_from_sim no)
-		(at 89.916 18.034 0)
-		(effects
-			(font
-				(size 1.27 1.27)
-			)
-			(justify left top)
-		)
-	)
-	(text "DSM"
-		(exclude_from_sim no)
-		(at 89.916 56.134 0)
-		(effects
-			(font
-				(size 1.27 1.27)
-			)
-			(justify left bottom)
-		)
-	)
-	(text "MAIN 1 : PA0 : TIM5_CH1\nMAIN 2 : PA1 : TIM5_CH2\nMAIN 3 : PA2 : TIM5_CH3\nMAIN 4 : PA3 : TIM5_CH4\nMAIN 5 : PC6 : TIM3_CH1\nMAIN 6 : PC7 : TIM3_CH2\nMAIN 7 : PB0 : TIM3_CH3\nMAIN 8 : PB1 : TIM3_CH4"
-		(exclude_from_sim no)
-		(at 23.8641 18.0091 0)
-		(effects
-			(font
-				(size 1.27 1.27)
-			)
-			(justify left top)
-		)
-	)
-	(text "PWM RC OUT"
-		(exclude_from_sim no)
-		(at 23.8641 15.4691 0)
-		(effects
-			(font
-				(size 1.27 1.27)
-			)
-			(justify left bottom)
-		)
-	)
-	(text "AUX1 : PB7 : TIM4_CH1\nAUX2 : PE11 : TIM1_CH2\nAUX3 : PE13 : TIM1_CH3\nAUX4 : PE14 : TIM1_CH4\n\nRCIN : PPM/SBUS/SRXL2\nRSSI_IN : PC1 : ADC123_IN11"
-		(exclude_from_sim no)
-		(at 23.8641 35.7891 0)
-		(effects
-			(font
-				(size 1.27 1.27)
-			)
-			(justify left top)
-		)
-	)
-	(text "ZH 1.5mm 4P\n\nPA9 : USART1_TX (Half Duplex)"
-		(exclude_from_sim no)
-		(at 89.916 86.614 0)
-		(effects
-			(font
-				(size 1.27 1.27)
-			)
-			(justify left top)
-		)
-	)
 	(label "UART1_RX"
 		(at 129.54 31.75 0)
@@
 		)
 		(instances
-			(project ""
+			(project "STM32-FC"
 				(path "/8d4cc317-3933-4aa6-844b-8c5c635e89c7/77caf73d-b7f5-48a6-9de3-ef3df69ee7d9"
 					(reference "#PWR079")
@@
 		)
 		(instances
-			(project ""
+			(project "STM32-FC"
 				(path "/8d4cc317-3933-4aa6-844b-8c5c635e89c7/77caf73d-b7f5-48a6-9de3-ef3df69ee7d9"
 					(reference "#PWR075")
@@
 		)
 		(instances
-			(project ""
+			(project "STM32-FC"
 				(path "/8d4cc317-3933-4aa6-844b-8c5c635e89c7/77caf73d-b7f5-48a6-9de3-ef3df69ee7d9"
 					(reference "#PWR077")
@@
 		)
 		(instances
-			(project ""
+			(project "STM32-FC"
 				(path "/8d4cc317-3933-4aa6-844b-8c5c635e89c7/77caf73d-b7f5-48a6-9de3-ef3df69ee7d9"
 					(reference "#PWR078")
@@
 		)
 		(instances
-			(project ""
+			(project "STM32-FC"
 				(path "/8d4cc317-3933-4aa6-844b-8c5c635e89c7/77caf73d-b7f5-48a6-9de3-ef3df69ee7d9"
 					(reference "JP1")
@@
 		)
 		(instances
-			(project ""
+			(project "STM32-FC"
 				(path "/8d4cc317-3933-4aa6-844b-8c5c635e89c7/77caf73d-b7f5-48a6-9de3-ef3df69ee7d9"
 					(reference "#PWR081")
@@
 		)
 		(instances
-			(project ""
+			(project "STM32-FC"
 				(path "/8d4cc317-3933-4aa6-844b-8c5c635e89c7/77caf73d-b7f5-48a6-9de3-ef3df69ee7d9"
 					(reference "J6")
