File: STM32-FC/schematic/memory.kicad_sch (KiCad schematic)
At the start: 9 parts, among them J4 TF-06A, U5 W25X40CLUXIG

Commit message: schematic update
Other:
- title: Memory -> STM32 Flight Controller
