File: STM32-FC/schematic/sensors.kicad_sch (KiCad schematic)
At the start: 18 parts, among them J5 JST ZH 1.5mm 2P, U6 BMI323, U7 ICM-42688-P, U8 LIS2MDLTR, U9 LPS22HH

Commit message: schematic update
Other:
- title: Sensors -> STM32 Flight Controller
Changed lines of the file:
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@@
 (kicad_sch
-	(version 20231120)
+	(version 20250114)
 	(generator "eeschema")
-	(generator_version "8.0")
+	(generator_version "9.0")
 	(paper "A4")
 	(title_block
-		(title "Sensors")
-		(date "2025-02-08")
-		(rev "A")
+		(title "STM32 Flight Controller")
+		(date "2025-09-16")
+		(rev "v1.0.0")
 		(company "NARAE")
 		(comment 1 "INHA Univ. Areo-modelling Club")
 		(comment 2 "2024 Winter UAV Project ")
 	)
+	(rectangle
+		(start 125.73 91.44)
+		(end 204.47 152.4)
+		(stroke
+			(width 0)
+			(type dash)
+		)
+		(fill
+			(type none)
+		)
+	)
+	(rectangle
+		(start 22.86 12.7)
+		(end 123.19 88.9)
+		(stroke
+			(width 0)
+			(type dash)
+		)
+		(fill
+			(type none)
+		)
+	)
+	(rectangle
+		(start 22.86 91.44)
+		(end 123.19 152.4)
+		(stroke
+			(width 0)
+			(type dash)
+		)
+		(fill
+			(type none)
+		)
+	)
+	(text "Close to\npin 9"
+		(exclude_from_sim no)
+		(at 153.67 36.195 0)
+		(effects
+			(font
+				(size 1.27 1.27)
+			)
+			(justify right bottom)
+		)
+	)
+	(text "Magnetic Sensor"
+		(exclude_from_sim no)
+		(at 126.746 15.494 0)
+		(effects
+			(font
+				(size 1.27 1.27)
+			)
+			(justify left bottom)
+		)
+	)
+	(text "Barometeric Pressure Sensor"
+		(exclude_from_sim no)
+		(at 126.746 94.234 0)
+		(effects
+			(font
+				(size 1.27 1.27)
+			)
+			(justify left bottom)
+		)
+	)
+	(text "Battery Monitoring"
+		(exclude_from_sim no)
+		(at 208.026 15.494 0)
+		(effects
+			(font
+				(size 1.27 1.27)
+			)
+			(justify left bottom)
+		)
+	)
+	(text "Accelerometer/Gyroscope1"
+		(exclude_from_sim no)
+		(at 24.13 15.494 0)
+		(effects
+			(font
+				(size 1.27 1.27)
+			)
+			(justify left bottom)
+		)
+	)
+	(text "SPI3_SCK  : PB3\nSPI3_MISO : PB4\nSPI3_MOSI : PB5\n\nGYRO2_NSS : PE3"
+		(exclude_from_sim no)
+		(at 23.876 96.774 0)
+		(effects
+			(font
+				(size 1.27 1.27)
+			)
+			(justify left top)
+		)
+	)
+	(text "SPI1_SCK  : PA5\nSPI1_MISO : PA6\nSPI1_MOSI : PA7\n\nBARO_NSS : PE6\nBARO_INT : PE7"
+		(exclude_from_sim no)
+		(at 126.746 96.774 0)
+		(effects
+			(font
+				(size 1.27 1.27)
+			)
+			(justify left top)
+		)
+	)
+	(text "JST ZH 1.5mm 2P\n\nV_BATT : PC0 : ADC123_IN10"
+		(exclude_from_sim no)
+		(at 208.026 18.034 0)
+		(effects
+			(font
+				(size 1.27 1.27)
+			)
+			(justify left top)
+		)
+	)
+	(text "SPI1_SCK  : PA5\nSPI1_MISO : PA6\nSPI1_MOSI : PA7\n\nGYRO1_NSS : PE5"
+		(exclude_from_sim no)
+		(at 23.876 18.034 0)
+		(effects
+			(font
+				(size 1.27 1.27)
+			)
+			(justify left top)
+		)
+	)
+	(text "Accelerometer/Gyroscope2"
+		(exclude_from_sim no)
+		(at 24.13 94.234 0)
+		(effects
+			(font
+				(size 1.27 1.27)
+			)
+			(justify left bottom)
+		)
+	)
+	(text "Close to\npin 5 and 6"
+		(exclude_from_sim no)
+		(at 190.5 71.755 0)
+		(effects
+			(font
+				(size 1.27 1.27)
+			)
+			(justify left bottom)
+		)
+	)
+	(text "SPI3_SCK  : PB3\nSPI3_MISO : PB4\nSPI3_MOSI : PB5\n\nMAG_NSS : PE4"
+		(exclude_from_sim no)
+		(at 126.746 18.034 0)
+		(effects
+			(font
+				(size 1.27 1.27)
+			)
+			(justify left top)
+		)
+	)
 	(junction
 		(at 87.63 36.83)
@@
 		)
 	)
-	(rectangle
-		(start 125.73 91.44)
-		(end 204.47 152.4)
-		(stroke
-			(width 0)
-			(type dash)
-		)
-		(fill
-			(type none)
-		)
-	)
-	(rectangle
-		(start 22.86 12.7)
-		(end 123.19 88.9)
-		(stroke
-			(width 0)
-			(type dash)
-		)
-		(fill
-			(type none)
-		)
-	)
-	(rectangle
-		(start 22.86 91.44)
-		(end 123.19 152.4)
-		(stroke
-			(width 0)
-			(type dash)
-		)
-		(fill
-			(type none)
-		)
-	)
-	(text "Close to\npin 9"
-		(exclude_from_sim no)
-		(at 153.67 36.195 0)
-		(effects
-			(font
-				(size 1.27 1.27)
-			)
-			(justify right bottom)
-		)
-	)
-	(text "Magnetic Sensor"
-		(exclude_from_sim no)
-		(at 126.746 15.494 0)
-		(effects
-			(font
-				(size 1.27 1.27)
-			)
-			(justify left bottom)
-		)
-	)
-	(text "Barometeric Pressure Sensor"
-		(exclude_from_sim no)
-		(at 126.746 94.234 0)
-		(effects
-			(font
-				(size 1.27 1.27)
-			)
-			(justify left bottom)
-		)
-	)
-	(text "Battery Monitoring"
-		(exclude_from_sim no)
-		(at 208.026 15.494 0)
-		(effects
-			(font
-				(size 1.27 1.27)
-			)
-			(justify left bottom)
-		)
-	)
-	(text "Accelerometer/Gyroscope1"
-		(exclude_from_sim no)
-		(at 24.13 15.494 0)
-		(effects
-			(font
-				(size 1.27 1.27)
-			)
-			(justify left bottom)
-		)
-	)
-	(text "SPI3_SCK  : PB3\nSPI3_MISO : PB4\nSPI3_MOSI : PB5\n\nGYRO2_NSS : PE3"
-		(exclude_from_sim no)
-		(at 23.876 96.774 0)
-		(effects
-			(font
-				(size 1.27 1.27)
-			)
-			(justify left top)
-		)
-	)
-	(text "SPI1_SCK  : PA5\nSPI1_MISO : PA6\nSPI1_MOSI : PA7\n\nBARO_NSS : PE6\nBARO_INT : PE7"
-		(exclude_from_sim no)
-		(at 126.746 96.774 0)
-		(effects
-			(font
-				(size 1.27 1.27)
-			)
-			(justify left top)
-		)
-	)
-	(text "JST ZH 1.5mm 2P\n\nV_BATT : PC0 : ADC123_IN10"
-		(exclude_from_sim no)
-		(at 208.026 18.034 0)
-		(effects
-			(font
-				(size 1.27 1.27)
-			)
-			(justify left top)
-		)
-	)
-	(text "SPI1_SCK  : PA5\nSPI1_MISO : PA6\nSPI1_MOSI : PA7\n\nGYRO1_NSS : PE5"
-		(exclude_from_sim no)
-		(at 23.876 18.034 0)
-		(effects
-			(font
-				(size 1.27 1.27)
-			)
-			(justify left top)
-		)
-	)
-	(text "Accelerometer/Gyroscope2"
-		(exclude_from_sim no)
-		(at 24.13 94.234 0)
-		(effects
-			(font
-				(size 1.27 1.27)
-			)
-			(justify left bottom)
-		)
-	)
-	(text "Close to\npin 5 and 6"
-		(exclude_from_sim no)
-		(at 190.5 71.755 0)
-		(effects
-			(font
-				(size 1.27 1.27)
-			)
-			(justify left bottom)
-		)
-	)
-	(text "SPI3_SCK  : PB3\nSPI3_MISO : PB4\nSPI3_MOSI : PB5\n\nMAG_NSS : PE4"
-		(exclude_from_sim no)
-		(at 126.746 18.034 0)
-		(effects
-			(font
-				(size 1.27 1.27)
-			)
-			(justify left top)
-		)
-	)
 	(label "SS2_SPI_MOSI"
 		(at 62.23 171.45 180)
@@
 		)
 		(instances
-			(project ""
+			(project "STM32-FC"
 				(path "/8d4cc317-3933-4aa6-844b-8c5c635e89c7/2d70a10f-8989-40ff-9a87-2cfa97b94251"
 					(reference "#PWR069")
@@
 		)
 		(instances
-			(project ""
+			(project "STM32-FC"
 				(path "/8d4cc317-3933-4aa6-844b-8c5c635e89c7/2d70a10f-8989-40ff-9a87-2cfa97b94251"
 					(reference "#PWR065")
@@
 		)
 		(instances
-			(project ""
+			(project "STM32-FC"
 				(path "/8d4cc317-3933-4aa6-844b-8c5c635e89c7/2d70a10f-8989-40ff-9a87-2cfa97b94251"
 					(reference "#PWR059")
@@
 		)
 		(instances
-			(project ""
+			(project "STM32-FC"
 				(path "/8d4cc317-3933-4aa6-844b-8c5c635e89c7/2d70a10f-8989-40ff-9a87-2cfa97b94251"
 					(reference "#FLG04")
@@
 		)
 		(instances
-			(project ""
+			(project "STM32-FC"
 				(path "/8d4cc317-3933-4aa6-844b-8c5c635e89c7/2d70a10f-8989-40ff-9a87-2cfa97b94251"
 					(reference "#PWR063")
@@
 		)
 		(instances
-			(project ""
+			(project "STM32-FC"
 				(path "/8d4cc317-3933-4aa6-844b-8c5c635e89c7/2d70a10f-8989-40ff-9a87-2cfa97b94251"
 					(reference "#PWR068")
@@
 		)
 		(instances
-			(project ""
+			(project "STM32-FC"
 				(path "/8d4cc317-3933-4aa6-844b-8c5c635e89c7/2d70a10f-8989-40ff-9a87-2cfa97b94251"
 					(reference "U7")
@@
 		)
 		(instances
-			(project ""
+			(project "STM32-FC"
 				(path "/8d4cc317-3933-4aa6-844b-8c5c635e89c7/2d70a10f-8989-40ff-9a87-2cfa97b94251"
 					(reference "#PWR067")
