File: STM32-FC/io_GPS.kicad_sch (KiCad schematic)
At the start: 8 parts, among them J10 GH 1.25mm 10P, J11 GH 1.25mm 6P

Commit message: v1.0 rollback
Parts:
- renumbered J11 to J10, J10 to J9, R38 to R23, R39 to R24, R40 to R25, R41 to R26, R42 to R27, R43 to R28
Other:
- title: STM32 Flight Controller -> GPS
