File: STM32-FC/io_RC_INPUT.kicad_sch (KiCad schematic)
At the start: 13 parts, among them J6 PWM_Conn_3x14, J7 ZH 1.5mm 4P, J8 GH 1.25mm 4P, J9 ZH 1.5mm 3P, Q1 PMDPB30XN, U11 TMUX1104

Commit message: v1.0 rollback
Parts:
- removed J8: GH 1.25mm 4P, JST_GH:JST_GH_SM04B-GHS-TB_04x1.25mm_Angled, symbol Connector_Generic:Conn_01x04
- removed Q1: PMDPB30XN, Nexperia_SOT1118:Nexperia_SOT1118, symbol Nexperia_PMD:PMDPB30XN
- removed R31, R32, R34: 10k, Resistor_SMD:R_0402_1005Metric, symbol Device:R_Small_US
- removed U11: TMUX1104, Package_SON:USON-10_2.5x1.0mm_P0.5mm, symbol TMUX1104:TMUX1104
- added JP1: SolderJumper_2_Open, Jumper:SolderJumper-2_P1.3mm_Open_TrianglePad1.0x1.5mm, symbol Jumper:SolderJumper_2_Open
- added Q2: S9013, Package_TO_SOT_SMD:SOT-23-3, symbol Device:Q_NPN_BEC
- R21: renamed from R33; value 120 -> 1k; LCSC C25079 -> C11702
- R22: renamed from R35; value 1k -> 10k; LCSC C106235 -> C25531
- renumbered J9 to J7, J7 to J8, R36 to R19, R37 to R20
Connections:
- net +5V_PWM2 is gone; now on net +5V: J6.16 (5V_RCIN)
- net RCIN is gone; now on net PPM_IN: J6.14 (RCIN)
- net SBUS is gone; now on net PPM_IN: R21.1
- net +5V: no longer J6.18 (5V_RSSI)
- net GND: now also J6.18 (GND), Q2.2 (E); no longer J6.19 (GND)
- net PPM_IN: now also JP1.2 (B)
- net UART1_RX: now also Q2.3 (C)
- net UART1_TX: now also JP1.1 (A)
- net at R21.2: now also Q2.1 (B)
- net +3.3V renamed +3.3V_RC
- net +5V_PWM1 renamed +5V_PWM
Other:
- note removed: "CRSF"
- note removed: "SH 1.0mm 4P PA9 : USART1_TX PA10 : USART1_RX"
- title: STM32 Flight Controller -> RC_INPUT
- moved on the sheet: J7, J8, R19, R20, R21, R22
