File: STM32-FC/io_communication.kicad_sch (KiCad schematic)
At the start: 17 parts, among them J12 GH 1.25mm 6P, J13 GH 1.25mm 6P, J14 GH 1.25mm 4P, J15 GH 1.25mm 4P, J16 GH 1.25mm 4P, U12 ATA6561-GBQW, U13 ATA6561-GBQW

Commit message: v1.0 rollback
Parts:
- U10: renamed from U12; symbol ATA6561-GBQW:ATA6561-GBQW_Small -> ATA6561-GBQW:ATA6561-GBQW_2
- U11: renamed from U13; symbol ATA6561-GBQW:ATA6561-GBQW_Small -> ATA6561-GBQW:ATA6561-GBQW_2
- renumbered C32 to C31, C33 to C32, C34 to C33, C35 to C34, J12 to J11, J13 to J12, J14 to J13, J15 to J14, J16 to J15, R44 to R29, R45 to R30, R46 to R31, R47 to R32, R48 to R33, R49 to R34
Other:
- title: STM32 Flight Controller -> Communication
