File: STM32-FC/memory.kicad_sch (KiCad schematic)
At the start: 9 parts, among them J4 TF-06A, U6 W25X40CLUXIG

Commit message: v1.0 rollback
Parts:
- U5: renamed from U6; footprint W25X40CLUX:USON_LUXIG_TR_HandSolder -> W25X40CLUX:USON_LUXIG TR_WIN-L
- renumbered C20 to C19, C21 to C20, R23 to R11, R24 to R12, R25 to R13, R26 to R14, R27 to R15
Other:
- title: STM32 Flight Controller -> Memory
