File: STM32-FC/sensors.kicad_sch (KiCad schematic)
At the start: 20 parts, among them J5 JST ZH 1.5mm 2P, U10 LPS22HH, U7 BMI323, U8 ICM-42688-P, U9 LIS2MDLTR

Commit message: v1.0 rollback
Parts:
- removed C36, C37: 100nF, Capacitor_SMD:C_0402_1005Metric, symbol Device:C
- C22: renamed from C23; value 100nF -> 100pF
- C24: renamed from C25; value 2.2uF -> 2.2nF
- C26: renamed from C27; LCSC C307423 -> C368809
- C27: renamed from C28; LCSC C307415 -> C77000
- R18: renamed from R30; LCSC C106235 -> C11702
- U6: renamed from U7; footprint BMI323 -> BMI323:BMI323_L; symbol BMI323:BMI323_Small -> BMI323:BMI323; Height 0.87 -> (none); Manufacturer_Name BOSCH -> (none); Manufacturer_Part_Number BMI323 -> (none); Mouser Part Number 262-BMI323 -> (none); Mouser Price/Stock https://www.mouser.co.uk/ProductDetail/Bosch-Sensortec/BMI3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 -> (none)
- U7: renamed from U8; symbol ICM-42688-P:ICM-42688-P_Small -> ICM-42688-P:ICM-42688-P_COMPACT
- U8: renamed from U9; symbol LIS2MDLTR:LIS2MDLTR_Small -> LIS2MDLTR:LIS2MDLTR
- U9: renamed from U10; footprint Package_LGA:ST_HLGA-10_2x2mm_P0.5mm_LayoutBorder3x2y -> LPS22HH:ST_HLGA-10_2x2mm_P0.5mm_LayoutBorder3x2y
- renumbered C22 to C21, C24 to C23, C26 to C25, C29 to C28, C30 to C29, C31 to C30, R28 to R16, R29 to R17
Connections:
- net MAG_C1: now reaches C30.1, U8.5 (C1)
- net GYRO1_INT: no longer names the net of U7.4 (INT1/INT)
- net GYRO2_INT: no longer names the net of U6.4 (INT1)
- no-connect marks 7 -> 9
Other:
- note added: "Close to pin 5 and 6"
- note added: "Close to pin 9"
- title: STM32 Flight Controller -> Sensors
- moved on the sheet: C21, C22, C23, C24, C25, C26, C27, C28, C29, C30, J5, R16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
