File: STM32-FC/usb.kicad_sch (KiCad schematic)
At the start: 28 parts, among them J2 USB_C_USB2.0_14P, J3 GH 1.25mm 6P, Q2 PMDPB30XN, Q3 PMDPB55XP, U2 USBLC6-2SC6, U3 TPS62840, U5 TPS62840

Commit message: v1.0 rollback
Parts:
- removed C19: 10uF, Capacitor_SMD:C_0402_1005Metric, symbol Device:C_Small
- removed D6: B5819W, Diode_SMD:D_SOD-323, symbol Device:D_Schottky_Small
- removed L1, L3: 2.2u, VLS201610ET-2R2M:VLS201610ET-2R2M, symbol Device:L_Iron_Small
- removed Q2: PMDPB30XN, Nexperia_SOT1118:Nexperia_SOT1118, symbol Nexperia_PMD:PMDPB30XN
- removed Q3: PMDPB55XP, Nexperia_SOT1118:Nexperia_SOT1118, symbol Nexperia_PMD:PMDPB55XPA
- removed R10, R9: 120, Resistor_SMD:R_0402_1005Metric, symbol Device:R_Small_US
- removed R11, R12: 10k, Resistor_SMD:R_0402_1005Metric, symbol Device:R_Small_US
- removed R14: 5k1, Resistor_SMD:R_0402_1005Metric, symbol Device:R_US
- removed R15, R16, R17, R18: 1k, Resistor_SMD:R_0402_1005Metric, symbol Device:R_Small_US
- removed R20, R22: 267k, Resistor_SMD:R_0402_1005Metric, symbol Device:R_Small_US
- removed U3, U5: TPS62840, Package_BGA:Texas_DSBGA-6_0.855x1.255mm_Layout2x3_P0.4mm_LevelC, symbol TPS62840:TPS62840YBG
- added C14, C18: 10uF, Capacitor_SMD:C_0402_1005Metric, symbol Device:C_Small
- added C15: 100nF, Capacitor_SMD:C_0402_1005Metric, symbol Device:C_Small
- added U3, U4: AMS1117-3.3, Package_TO_SOT_SMD:SOT-89-3, symbol Regulator_Linear:AMS1117-3.3
- C13: renamed from C14; value 4.7uF -> 10uF; LCSC C307423 -> C77000
- C16: value 4.7uF -> 100nF; LCSC C307423 -> C1525
- C17: LCSC C307415 -> C77000
- renumbered D5 to D6, R19 to R10, R13 to R9
Connections:
- net +3.3V: now also C15.1, U3.2 (VO)
- net +5V: now also J3.1 (Pin_1), J3.2 (Pin_2), C14.1, U3.3 (VI), U4.3 (VI); no longer C16.1
- net GND: now also U2.2 (GND), C14.2, C15.2, C18.2, U3.1 (GND), U4.1 (GND)
- net USB_CONN_D+: now also U2.3 (I/O2)
- net USB_CONN_D-: now also U2.1 (I/O1)
- net USB_D+: now also U2.4 (I/O2)
- net USB_D-: now also U2.6 (I/O1)
- net VBUS: now also U2.5 (VBUS)
- net at J2.B5 (CC2): now also J2.A5 (CC1), R9.1
- new net +3.3V_RC: C16.1, C18.1, U4.2 (VO)
Other:
- note removed: "3.3V for IMUs with Power Gating"
- note removed: "PE15 : PWR_SEL0 PA15 : PWR_SEL1"
- note removed: "POWER MOSFET"
- title: STM32 Flight Controller -> USB & POWER
- moved on the sheet: C13, C17, J3
