File: STM32-FC/STM32-FC.kicad_sch (KiCad schematic)
At the start: 35 parts, among them J1 GH 1.25mm 6P, Q1 PMDPB30XN, U1 STM32F407VETx, Y1 16MHz

Commit message: v1.0 rollback
Parts:
- removed C15: 100nF, Capacitor_SMD:C_0402_1005Metric, symbol Device:C_Small
- removed Q1: PMDPB30XN, Nexperia_SOT1118:Nexperia_SOT1118, symbol Nexperia_PMD:PMDPB30XN
- removed R5: 10k, Resistor_SMD:R_0402_1005Metric, symbol Device:R_Small_US
- added D1: White, LED_SMD:LED_0402_1005Metric, symbol Device:LED_Small
- added Q1: S9013, Package_TO_SOT_SMD:SOT-23-3, symbol Device:Q_NPN_BEC
- added R4: 1k, Resistor_SMD:R_0402_1005Metric, symbol Device:R_Small_US
- added SW2: SW_DIP_x03, Button_Switch_SMD:SW_DIP_SPSTx03_Slide_KingTek_DSHP03TJ_W5.25mm_P1.27mm_JPin, symbol Switch:SW_DIP_x03
- added TP1, TP2, TP3: Test Pin, Connector_PinHeader_1.27mm:PinHeader_1x03_P1.27mm_Vertical, symbol Connector:Conn_01x03_Socket
- C2: value 4.7uF -> 10uF; LCSC C307415 -> C77000
- D5: renamed from D4; value Green -> Blue; LCSC C130722 -> C130724
- R1: renamed from R2; value 10k -> 100k; LCSC C25531 -> C25741
- R2: renamed from R1; value 10k -> 100k; LCSC C25531 -> C25741
- R3: value 120 -> 4k7; LCSC C25079 -> C25900
- R5: renamed from R4; value 120 -> 180; LCSC C25079 -> C38941
- R6, R7, R8: value 120 -> 1k; LCSC C25079 -> C11702
- renumbered C11 to C10, C12 to C11, C13 to C12, C5 to C35, C6 to C5, C7 to C6, C8 to C7, C9 to C8, C10 to C9, D1 to D3, D3 to D4
Connections:
- net +3.3V: now also D1.2 (A), SW2.2, SW2.3
- net +5V: now also SW2.6
- net BOOT0: now also R1.2, SW2.4; no longer J1.5 (Pin_5), R1.1
- net GND: now also R1.1, R2.1, Q1.2 (E), R4.2; no longer R1.2, R2.2
- net SPI1_MISO: now also TP2.2 (Pin_2)
- net SPI1_MOSI: now also TP2.3 (Pin_3)
- net SPI1_SCK: now also TP2.1 (Pin_1)
- net SPI2_MISO: now also TP1.2 (Pin_2)
- net SPI2_MOSI: now also TP1.3 (Pin_3)
- net SPI2_SCK: now also TP1.1 (Pin_1)
- net SPI3_MISO: now also TP3.2 (Pin_2)
- net SPI3_MOSI: now also TP3.3 (Pin_3)
- net SPI3_SCK: now also TP3.1 (Pin_1)
- net at BZ1.2 (+), D3.2 (A): now also Q1.3 (C)
- net BOOT1: now reaches U1.37 (PB2)
- net BOOT1: now also R2.2, SW2.5; no longer R2.1
- net at R5.2: now also Q1.1 (B)
- net GYRO1_INT: no longer names the net of U1.39 (PE8)
- net GYRO2_INT: no longer names the net of U1.8 (PC14)
- net LED_GREEN renamed LED_BLUE
- net PWR_SEL0: no longer names the net of U1.46 (PE15)
- net PWR_SEL1: no longer names the net of U1.77 (PA15)
- net RC_PPM renamed PPM_IN
- net RC_RX renamed DSM/SBUS
- net RC_SEL0: no longer names the net of U1.41 (PE10)
- net RC_SEL1: no longer names the net of U1.40 (PE9)
- net RC_TX renamed SRXL2
- net SW_PWR_IMU: no longer names the net of U1.43 (PE12)
- new net: D1.1 (K), R4.1
- new net +5V_PWM: SW2.1
- no-connect marks 1 -> 9
Other:
- sheet RC_INPUT ports: added none; removed RC_SEL0, RC_SEL1
- sheet Sensors ports: added none; removed GYRO1_INT, GYRO2_INT
- sheet USB & POWER ports: added none; removed PWR_SEL0, PWR_SEL1, SW_PWR_IMU
- note added: "- Boot |X|0| : Main Flash |0|1| : System FLASH |1|1| : SRAM - PWR Select Switch to set power supplied from BEC to be supplied to the board"
- note added: "Boot & 5V PWR Select"
- note added: "W : PWR R : PE0 Y : PE1 B : PE2"
- note removed: "W : PA4 R : PE0 Y : PE1 B : PE2"
- moved on the sheet: BZ1, C1, C10, C11, C12, C2, C3, C35, C4, C5, C6, C7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

Commit message: schematic update
Other:
- sheet Communication: file io_communication.kicad_sch -> schematic/io_communication.kicad_sch
- sheet GPS: file io_GPS.kicad_sch -> schematic/io_GPS.kicad_sch
- sheet Memory: file memory.kicad_sch -> schematic/memory.kicad_sch
- sheet RC_INPUT: file io_RC_INPUT.kicad_sch -> schematic/io_RC_INPUT.kicad_sch
- sheet Sensors: file sensors.kicad_sch -> schematic/sensors.kicad_sch
- sheet USB & POWER: file usb.kicad_sch -> schematic/usb.kicad_sch
