File: STM32-FC/STM32-FC.kicad_pcb (KiCad board)
At the start: 4 copper layers, 39 x 48.5 mm, 129 parts, among them J1 GH 1.25mm 6P, J10 GH 1.25mm 10P, J11 GH 1.25mm 6P, J12 GH 1.25mm 6P, J13 GH 1.25mm 6P, J14 GH 1.25mm 4P, J15 GH 1.25mm 4P, J16 GH 1.25mm 4P, J2 USB_C_USB2.0_14P, J3 GH 1.25mm 6P, J4 TF-06A, J5 JST ZH 1.5mm 2P, J6 PWM_Conn_3x14, J7 ZH 1.5mm 4P, J8 GH 1.25mm 4P, J9 ZH 1.5mm 3P, Q1 PMDPB30XN, Q2 PMDPB30XN, Q3 PMDPB55XP, U1 STM32F407VETx, U10 LPS22HH, U11 TMUX1104, U12 ATA6561-GBQW, U13 ATA6561-GBQW, U2 USBLC6-2SC6, U3 TPS62840, U5 TPS62840, U6 W25X40CLUXIG, U7 BMI323, U8 ICM-42688-P, U9 LIS2MDLTR, Y1 16MHz

Commit message: v1.0 rollback
Parts:
- removed the C19 at (140.5, 106.5)
- removed C36, C37: 100nF, Capacitor_SMD:C_0402_1005Metric
- removed the D6 at (126.5, 76.8)
- removed the J8 at (155.4, 98.6)
- removed L1, L3: 2.2u, VLS201610ET-2R2M:VLS201610ET-2R2M
- removed Q3: PMDPB55XP, Nexperia_SOT1118:Nexperia_SOT1118
- removed the R10 at (148.9, 103.2)
- removed the R11 at (144.4, 103.2)
- removed the R12 at (149.9, 103.2)
- removed the R14 at (129.8, 88.5)
- removed the R15 at (144.9, 106.2)
- removed the R16 at (149.4, 105.2)
- removed the R17 at (149.4, 106.2)
- removed the R18 at (144.9, 105.2)
- removed the R20 at (135.8, 102.8)
- removed the R22 at (141.0, 102.8)
- removed the R31 at (106.2, 94.2)
- removed the R32 at (106.2, 95.2)
- removed the R34 at (132.7, 81.2)
- removed the R5 at (133.0, 77.8)
- removed the R9 at (145.4, 103.2)
- removed the U11 at (103.7, 94.8)
- removed the U5 at (140.5, 104.5)
- added C14: 10uF, Capacitor_SMD:C_0402_1005Metric, B.Cu at (135.0, 106.4)
- added C18: 10uF, Capacitor_SMD:C_0402_1005Metric, B.Cu at (132.5, 102.0)
- added D1: White, LED_SMD:LED_0402_1005Metric, F.Cu at (146.2, 104.2)
- added JP1: SolderJumper_2_Open, Jumper:SolderJumper-2_P1.3mm_Open_TrianglePad1.0x1.5mm, F.Cu at (123.5, 116.4)
- added R4: 1k, Resistor_SMD:R_0402_1005Metric, F.Cu at (148.2, 104.2)
- added SW2: SW_DIP_x03, Button_Switch_SMD:SW_DIP_SPSTx03_Slide_KingTek_DSHP03TJ_W5.25mm_P1.27mm_JPin, B.Cu at (154.0, 99.2)
- added TP1: Test Pin, Connector_PinHeader_1.27mm:PinHeader_1x03_P1.27mm_Vertical, B.Cu at (147.0, 95.4)
- added TP2: Test Pin, Connector_PinHeader_1.27mm:PinHeader_1x03_P1.27mm_Vertical, B.Cu at (143.2, 104.3)
- added TP3: Test Pin, Connector_PinHeader_1.27mm:PinHeader_1x03_P1.27mm_Vertical, B.Cu at (147.0, 98.6)
- added U4: AMS1117-3.3, Package_TO_SOT_SMD:SOT-89-3, B.Cu at (136.0, 103.0)
- C1, C3, C4, Y1: moved to F.Cu
- C10: renamed from C11; moved to F.Cu
- C13: renamed from C14; value 4.7uF -> 10uF
- C16: value 4.7uF -> 100nF
- C2: value 4.7uF -> 10uF; moved to F.Cu
- C22: renamed from C23; value 100nF -> 100pF
- C24: renamed from C25; value 2.2uF -> 2.2nF
- C35: renamed from C5; moved to F.Cu
- C7: renamed from C8; moved to F.Cu
- C8: renamed from C9; moved to F.Cu
- C9: renamed from C10; moved to F.Cu
- D5: renamed from D4; value Green -> Blue
- Q1: value PMDPB30XN -> S9013; footprint Nexperia_SOT1118:Nexperia_SOT1118 -> Package_TO_SOT_SMD:SOT-23-3
- Q2: value PMDPB30XN -> S9013; footprint Nexperia_SOT1118:Nexperia_SOT1118 -> Package_TO_SOT_SMD:SOT-23-3; moved to F.Cu
- R1: renamed from R2; value 10k -> 100k
- R2: renamed from R1; value 10k -> 100k; moved to B.Cu
- R21: renamed from R33; value 120 -> 1k
- R22: renamed from R35; value 1k -> 10k
- R3: value 120 -> 4k7; moved to F.Cu
- R5: renamed from R4; value 120 -> 180
- R6, R7, R8: value 120 -> 1k
- U3: value TPS62840 -> AMS1117-3.3; footprint Package_BGA:Texas_DSBGA-6_0.855x1.255mm_Layout2x3_P0.4mm_LevelC -> Package_TO_SOT_SMD:SOT-89-3
- moved R2 26.0 mm to (154.6, 94.5)
- moved R20 25.0 mm to (127.2, 104.0), turned to -90 degrees
- moved C12 23.4 mm to (142.0, 80.5), turned to 180 degrees
- moved R22 23.1 mm to (132.8, 102.5), turned to -90 degrees
- moved C35 23.0 mm to (134.1, 97.8), turned to 180 degrees
- moved C11 21.6 mm to (142.0, 81.5), turned to 180 degrees
- moved R21 20.5 mm to (127.2, 102.0), turned to 90 degrees
- moved C15 20.3 mm to (132.5, 104.0), turned to 0 degrees
- moved Q2 17.1 mm to (130.0, 103.0), turned to 0 degrees
- moved C3 16.9 mm to (133.5, 95.2)
- moved C10 14.4 mm to (131.6, 96.2), turned to 0 degrees
- moved C9 10.1 mm to (131.6, 95.2), turned to 0 degrees
- moved C7 8.10 mm to (133.5, 94.2), turned to 180 degrees
- moved C8 7.38 mm to (131.6, 94.2)
- moved Y1 7.24 mm to (136.8, 103.6)
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- renumbered C12 to C11, C13 to C12, C20 to C19, C21 to C20, C22 to C21, C24 to C23, C26 to C25, C27 to C26, C28 to C27, C29 to C28, C30 to C29, C31 to C30, C32 to C31, C33 to C32, C34 to C33, C35 to C34, C6 to C5, C7 to C6, D1 to D3, D3 to D4, D5 to D6, J11 to J10, J12 to J11, J13 to J12, J14 to J13, J15 to J14, J16 to J15, J9 to J7, J7 to J8, J10 to J9, R19 to R10, R23 to R11, R24 to R12, R25 to R13, R26 to R14, R27 to R15, R28 to R16, R29 to R17, R30 to R18, R36 to R19, R37 to R20, R38 to R23, R39 to R24, R40 to R25, R41 to R26, R42 to R27, R43 to R28, R44 to R29, R45 to R30, R46 to R31, R47 to R32, R48 to R33, R49 to R34, R13 to R9, U12 to U10, U13 to U11, U6 to U5, U7 to U6, U8 to U7, U9 to U8, U10 to U9
Connections:
- net /LED_GREEN renamed /LED_BLUE
- net /RC_TX renamed /UART1_TX
- net Net-(U9-C1) renamed /Sensors/MAG_C1
- C16 pad 1: +5V -> +3.3V_RC
- J1 pad 5: /BOOT0 -> unconnected-(J1-Pin_5-Pad5)
- J2 pad B5: Net-(J2-CC2) -> Net-(J2-CC1)
- J3 pad 1: Net-(D6-A) -> +5V
- J3 pad 2: Net-(D6-A) -> +5V
- J6 pad 14: /RC_INPUT/RCIN -> /TIM1_CH4
- J6 pad 15: +5V_PWM1 -> +5V_PWM
- J6 pad 16: +5V_PWM2 -> +5V
- J6 pad 18: +5V -> GND
- J7 pad 1: +3.3V -> +3.3V_RC
- J7 pad 3: /RC_RX -> /UART1_RX
- Q1 pad 1: GND -> Net-(Q1-B)
- Q1 pad 2: Net-(Q1A-G) -> GND
- Q1 pad 3: /RC_RX -> Net-(BZ1-+)
- Q2 pad 1: GND -> Net-(Q2-B)
- Q2 pad 2: Net-(Q2A-G) -> GND
- Q2 pad 3: Net-(Q3B-G) -> /UART1_RX
- R1 pad 1: /BOOT0 -> GND
- R1 pad 2: GND -> /BOOT0
- R19 pad 1: +3.3V -> +3.3V_RC
- R19 pad 2: /RC_RX -> /UART1_RX
- R2 pad 1: Net-(U1-PB2) -> GND
- R2 pad 2: GND -> /BOOT1
- R20 pad 1: /RC_PPM -> /TIM1_CH4
- R21 pad 1: /RC_INPUT/SBUS -> /TIM1_CH4
- R21 pad 2: Net-(Q1B-G) -> Net-(Q2-B)
- R22 pad 1: +3.3V -> +3.3V_RC
- R22 pad 2: /RC_RX -> /UART1_RX
- R5 pad 2: Net-(Q1A-G) -> Net-(Q1-B)
- U1 pad 37: Net-(U1-PB2) -> /BOOT1
- U1 pad 39: /GYRO1_INT -> unconnected-(U1-PE8-Pad39)
- U1 pad 40: /RC_SEL1 -> unconnected-(U1-PE9-Pad40)
- U1 pad 41: /RC_SEL0 -> unconnected-(U1-PE10-Pad41)
- U1 pad 43: /SW_PWR_IMU -> unconnected-(U1-PE12-Pad43)
- U1 pad 45: /RC_PPM -> /TIM1_CH4
- U1 pad 46: /PWR_SEL0 -> unconnected-(U1-PE15-Pad46)
- U1 pad 69: /RC_RX -> /UART1_RX
- U1 pad 77: /PWR_SEL1 -> unconnected-(U1-PA15-Pad77)
- U1 pad 8: /GYRO2_INT -> unconnected-(U1-PC14-Pad8)
- U6 pad 4: /GYRO2_INT -> unconnected-(U6-INT1-Pad4)
- U7 pad 4: /GYRO1_INT -> unconnected-(U7-INT1/INT-Pad4)
Routing:
- net GND: track 11.2 -> 169.1 mm, vias 1 -> 41
- net /UART1_RX: track 0.00 -> 119.1 mm, vias 0 -> 3
- net +3.3V: track 18.9 -> 130.5 mm, vias 2 -> 24
- net /UART1_TX: track 0.00 -> 79.7 mm, vias 0 -> 1
- net /UART5_TX: track 0.00 -> 62.3 mm, vias 0 -> 2
- net /UART5_RX: track 0.00 -> 56.6 mm, vias 0 -> 2
- net +3.3V_RC: track 0.00 -> 54.9 mm, vias 0 -> 3
- net +5V: track 0.00 -> 53.2 mm, vias 0 -> 16
- net /TIM1_CH4: track 0.00 -> 52.9 mm, vias 0 -> 2
- net +5V_PWM: track 0.00 -> 40.1 mm, vias 0 -> 1
- net /TIM3_CH1: track 0.00 -> 39.3 mm, vias 0 -> 1
- net /SPI2_MOSI: track 0.00 -> 38.8 mm, vias 0 -> 2
- net /TIM3_CH2: track 0.00 -> 37.5 mm, vias 0 -> 1
- net /TIM4_CH4: track 0.00 -> 36.6 mm, vias 0 -> 1
- net /BOOT1: track 0.00 -> 35.5 mm, vias 0 -> 2
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Other:
- board text added: "NARAE STM32 FC"
- board text added: "SPI1"
- board text added: "SPI2"
- board text added: "SPI3"
- board text removed: "CRSF"
- board text removed: "NARAE STM32 FC v2"
