File: DevTool/DevTool.kicad_pcb (KiCad board)
At the start: 2 copper layers, 50.8 x 57.2 mm, 25 parts, among them J1 2.54mm 3P, J10 2.54mm 6P, J11 2.54mm 4P, J12 GH 1.25mm 6P, J13 ZH 1.5mm 3P, J14 ZH 1.5mm 4P, J15 GH 1.25mm 4P, J16 GH 1.25mm 6P, J17 2.54mm 3P, J18 2.54mm 4P, J19 2.54mm 4P, J2 GH 1.25mm 6P, J20 2.54mm 6P, J21 ZH 1.5mm 3P, J22 GH 1.25mm 4P, J23 ZH 1.5mm 4P, J3 GH 1.25mm 4P, J4 GH 1.25mm 6P, J5 GH 1.25mm 4P, J6 GH 1.25mm 6P, J7 GH 1.25mm 4P, J8 JTAG 20 Pin, J9 GH 1.25mm 4P, SW1 SW_Push

Commit message: update : Development board
Parts:
- removed J13, J21: ZH 1.5mm 3P, JST_ZH:JST_ZH_S3B-ZR-SM4A-TF_1x03-1MP_P1.50mm_Horizontal
- removed J17: 2.54mm 3P, Connector_PinHeader_2.54mm:PinHeader_1x03_P2.54mm_Vertical
- removed J8: JTAG 20 Pin, Connector_IDC:IDC-Header_2x10_P2.54mm_Vertical
- J1: value 2.54mm 3P -> 2.54mm 6P; footprint Connector_PinHeader_2.54mm:PinHeader_1x03_P2.54mm_Vertical -> Connector_PinHeader_2.54mm:PinHeader_1x06_P2.54mm_Vertical
- J14, J23: moved to F.Cu
- moved J23 23.8 mm to (152.5, 83.5), turned to 90 degrees
- moved J2 19.6 mm to (116.5, 82.0)
- moved J1 11.6 mm to (122.5, 90.6)
- moved J11 8.52 mm to (127.5, 102.7)
- moved J3 8.52 mm to (153.5, 106.5)
- moved J5 8.52 mm to (146.5, 106.5)
- moved J7 8.52 mm to (139.5, 106.5)
- moved J9 8.52 mm to (132.5, 106.5)
- moved C1 8.05 mm to (116.5, 74.0)
- moved SW1 8.05 mm to (116.5, 68.0)
- moved J18 6.04 mm to (147.0, 87.3), turned to 180 degrees
- moved J14 3.66 mm to (152.5, 93.5), turned to 90 degrees
Connections:
- C1 pad 1: /BOOT0 -> /NRST
- J1 pad 1: unconnected-(J1-Pin_1-Pad1) -> +3.3V
- J1 pad 2: /BOOT0 -> /SWDIO
- J1 pad 3: +3.3V -> /SWCLK
- J2 pad 5: /BOOT0 -> unconnected-(J2-Pin_5-Pad5)
- SW1 pad 2: /BOOT0 -> /NRST
Routing:
- net +3.3V: track 52.8 -> 7.25 mm
- net /BOOT0: track 31.1 -> 0.00 mm
- net /NRST: track 10.1 -> 27.3 mm
- net /UART1_RX: track 14.9 -> 0.00 mm
- net +5V: track 127.5 -> 142.2 mm, vias 1 -> 0
- net /SWDIO: track 17.4 -> 6.86 mm
- net /SWCLK: track 16.3 -> 6.12 mm
- net GND: track 67.1 -> 59.6 mm, vias 0 -> 5
- net /UART1_TX: track 16.0 -> 15.3 mm
- net unconnected-(J2-Pin_5-Pad5): track 0.00 -> 0.60 mm
Other:
- board size 50.8 x 57.2 mm -> 45 x 55.5 mm
- board text added: "* 3.3V: Output Only"
- board text added: "3.3V*"
- board text added: "GPS"
- board text added: "N.C."
- board text added: "NARAEON DEV BOARD"
- board text added: "NARAEON Development Board v1.1 NARAE, INHA University, Korea."
- board text added: "NRST"
- board text added: "SRXL2"
- board text added: "STLink"
- board text added: "SWCLK"
- board text added: "SWDIO"
- board text added: "Upload & Debugging: - Connect STLink → 'STLink' pinheader. - Connect FC → 'DEBUG' port. Module Test (ex. GPS): - Connect the 'GPS' port to the module (e.g., GPS) and the FC. - Probe the pinheader with a logic analyzer or oscilloscope to verify signals"
- board text removed: "0"
- board text removed: "1"
- board text removed: "3.3V"
- board text removed: "BOOT0"
- board text removed: "DSM*"
- board text removed: "GPS 2nd"
- board text removed: "I2C/CAN"
- board text removed: "SRXL2*"
