File: DevTool/DevTool.kicad_sch (KiCad schematic)
At the start: 25 parts, among them J1 2.54mm 3P, J10 2.54mm 6P, J11 2.54mm 4P, J12 GH 1.25mm 6P, J13 ZH 1.5mm 3P, J14 ZH 1.5mm 4P, J15 GH 1.25mm 4P, J16 GH 1.25mm 6P, J17 2.54mm 3P, J18 2.54mm 4P, J19 2.54mm 4P, J2 GH 1.25mm 6P, J20 2.54mm 6P, J21 ZH 1.5mm 3P, J22 GH 1.25mm 4P, J23 ZH 1.5mm 4P, J3 GH 1.25mm 4P, J4 GH 1.25mm 6P, J5 GH 1.25mm 4P, J6 GH 1.25mm 6P, J7 GH 1.25mm 4P, J8 JTAG 20 Pin, J9 GH 1.25mm 4P, SW1 SW_Push

Commit message: update : Development board
Parts:
- removed J1, J17: 2.54mm 3P, Connector_PinHeader_2.54mm:PinHeader_1x03_P2.54mm_Vertical, symbol Connector:Conn_01x03_Pin
- removed J13, J21: ZH 1.5mm 3P, JST_ZH:JST_ZH_S3B-ZR-SM4A-TF_1x03-1MP_P1.50mm_Horizontal, symbol Connector_Generic:Conn_01x03
- removed J8: JTAG 20 Pin, Connector_IDC:IDC-Header_2x10_P2.54mm_Vertical, symbol Connector:Conn_ARM_JTAG_SWD_20
- added J1: 2.54mm 6P, Connector_PinHeader_2.54mm:PinHeader_1x06_P2.54mm_Vertical, symbol Connector:Conn_01x06_Pin
Connections:
- net +3.3V: now also J1.1 (Pin_1)
- net GND: now also J1.6 (Pin_6)
- net NRST: now also C1.1, SW1.2, J1.4 (Pin_4)
- net SWCLK: now also J1.3 (Pin_3)
- net SWDIO: now also J1.2 (Pin_2)
- removed net BOOT0: C1.1, J2.5 (Pin_5), SW1.2
- no-connect marks 12 -> 5
Other:
- note removed: "DSM"
- note removed: "For Rev. 2"
- note removed: "ZH 1.5mm 3P PA10 : USART1_RX"
- company: (none) -> NARAE, INHA University
- title: (none) -> NARAEON Development Board
- moved on the sheet: J10, J11, J12, J14, J15, J16, J18, J19, J20, J22, J23, J3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
